File: hardware/pcb/stratolink.kicad_sch (KiCad schematic)
At the start: 61 parts, among them J1 Conn_Header_JST_PH_1x02_P2mm_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, J2 Conn_Header_JST_PH_1x02_P2mm_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, J20 Conn_ARM_SWD_TagConnect_TC203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, J3 Conn_PinHeader_1x07_P2.54mm_V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, J4 Conn_PinHeader_1x07_P2.54mm_V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, U2 RAK3172, U5 TMP117NAIYBGR, U7 LIS2DH12TR

Commit message: [PROD] Stratolink Pico Mainboard V1
Parts:
- added D1: ESD9B3.3ST5G, Diode_SMD:D_SOD-523, symbol Diode:ESD9B3.3ST5G
- renumbered R17 to FB1
Connections:
- net GND: now also J3.4 (Pin_4), J4.1 (Pin_1), U1.17 (NC), U1.21 (EP), U1.9 (NC), D1.1 (A1)
- net PB5: no longer J3.4 (Pin_4)
- net RSTN: no longer J4.1 (Pin_1)
- net at AE1.1 (A), U2.12 (RF): now also D1.2 (A2)
- net at C10.1, FB1.1, R18.1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: now also U3.6 (V_BCKP)
