File: hardware/pcb/stratolink.kicad_sch (KiCad schematic)
At the start: 62 parts, among them J1 Conn_Header_JST_PH_1x02_P2mm_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, J2 Conn_Header_JST_PH_1x02_P2mm_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, J20 Conn_ARM_SWD_TagConnect_TC203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, J3 Conn_PinHeader_1x07_P2.54mm_V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, J4 Conn_PinHeader_1x07_P2.54mm_V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, U2 RAK3172, U5 TMP117NAIYBGR, U7 LIS2DH12TR

Commit message: hardware: start v1.1 with corrected TMP117 symbol and routing
Use hardware/pcb as the canonical working project. Preserve component placement, correct the DSBGA ball map and local copper, add the v1.1/v2 checklist and canonical-path verification records. PCB saved in KiCad 10 format.
Parts:
- U5: Description_1 0.1°C digital temperature sensor, 48-bit EEPROM, PT100/PT10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 -> TMP117N precision digital temperature sensor; +/-0.2 C from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
Connections:
- net +3.3V: now also U5.B1 (V+); no longer U5.C1 (V+)
- net GND: now also U5.C1 (ADD0), U5.C2 (ALERT); no longer U5.A2 (GND), U5.B1 (ALERT)
- net SCL: now also U5.A2 (SCL); no longer U5.A1 (SCL)
- net SDA: now also U5.A1 (SDA); no longer U5.C2 (SDA)
Other:
- title: PICO Mainboard -> PICO Mainboard v1.1
Changed lines of the file:
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@@
 	(paper "User" 265 190)
 	(title_block
-		(title "PICO Mainboard")
-		(date "2026-02-08")
-		(rev "2026-02-08")
+		(title "PICO Mainboard v1.1")
+		(date "2026-10-12")
+		(rev "1.1")
 		(company "            Global pico-balloon telemetry system.")
 		(comment 1 "             Stratolink")
@@
 			)
 		)
-		(property "Datasheet" ""
+		(property "Datasheet" "https://www.ti.com/lit/ds/symlink/tmp117.pdf"
 			(at 38.1 160.02 0)
 			(effects
@@
 			)
 		)
-		(property "Description" ""
+		(property "Description" "TMP117N precision digital temperature sensor; +/-0.2 C from -40 to 100 C; YBG DSBGA-6"
 			(at 38.1 160.02 0)
 			(effects
@@
 			)
 		)
-		(property "Description_1" "\n                        \n                            0.1°C digital temperature sensor, 48-bit EEPROM, PT100/PT1000 RTD replacement\n                        \n"
+		(property "Description_1" "TMP117N precision digital temperature sensor; +/-0.2 C from -40 to 100 C; YBG DSBGA-6"
 			(at 38.1 160.02 0)
 			(effects
@@
 			)
 		)
-		(pin "A1"
-		)
-		(pin "B1"
-		)
 		(pin "A2"
 		)
-		(pin "B2"
-		)
 		(pin "C2"
 		)
+		(pin "B2"
+		)
 		(pin "C1"
 		)
+		(pin "A1"
+		)
+		(pin "B1"
+		)
 		(instances

Commit message: hardware: remove microphone from v1.1 payload
Parts:
- removed C13: 100nF, Capacitor_SMD:C_0402_1005Metric, symbol Device:C
- removed MK1: T3902, lib:MIC_T3902, symbol T3902:T3902
- removed R20: 33Ω, Resistor_SMD:R_0402_1005Metric, symbol Device:R_US
Connections:
- net CLK: no longer names the net of U2.32 (PB3/ADC1)
- net PDM: no longer names the net of U2.31 (PB4/ADC2)
- no-connect marks 0 -> 2
Other:
- note removed: "Mic"
