File: hardware/pcb/stratolink.kicad_sch (KiCad schematic)
At the start: 59 parts, among them J1 Conn_Header_JST_PH_1x02_P2mm_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, J2 Conn_Header_JST_PH_1x02_P2mm_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, J20 Conn_ARM_SWD_TagConnect_TC203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, J3 Conn_PinHeader_1x07_P2.54mm_V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, J4 Conn_PinHeader_1x07_P2.54mm_V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, U2 RAK3172, U5 TMP117NAIYBGR, U7 LIS2DH12TR

Commit message: hardware: add v1.1 side solar solder mounts
Parts:
- J1: value Conn_Header_JST_PH_1x02_P2mm_Vertical_SMD -> Solar panel direct solder; footprint Connector_PinHeader_1.00mm:PinHeader_1x02_P1.00mm_Vertical -> lib:Solar_Notch_Right_1p0x1p5; now left out of the parts list
- J2: value Conn_Header_JST_PH_1x02_P2mm_Vertical_SMD -> Solar panel direct solder; footprint Connector_PinHeader_1.00mm:PinHeader_1x02_P1.00mm_Vertical -> lib:Solar_Notch_Left_1p0x1p5; now left out of the parts list
Changed lines of the file:
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@@
 		(unit 1)
 		(exclude_from_sim no)
-		(in_bom yes)
+		(in_bom no)
 		(on_board yes)
 		(dnp no)
@@
 			)
 		)
-		(property "Value" "Conn_Header_JST_PH_1x02_P2mm_Vertical_SMD"
+		(property "Value" "Solar panel direct solder"
 			(at 194.31 99.06 0)
 			(effects
@@
 			)
 		)
-		(property "Footprint" "Connector_PinHeader_1.00mm:PinHeader_1x02_P1.00mm_Vertical"
+		(property "Footprint" "lib:Solar_Notch_Right_1p0x1p5"
 			(at 194.31 105.41 0)
 			(effects
@@
 			)
 		)
-		(property "Datasheet" "https://www.jst-mfg.com/product/pdf/eng/ePH.pdf"
+		(property "Datasheet" ""
 			(at 194.31 105.41 0)
 			(effects
@@
 			)
 		)
-		(property "Description" "Male JST PH 2 pin connector"
+		(property "Description" ""
 			(at 194.31 105.41 0)
 			(effects
@@
 		(unit 1)
 		(exclude_from_sim no)
-		(in_bom yes)
+		(in_bom no)
 		(on_board yes)
 		(dnp no)
@@
 			)
 		)
-		(property "Value" "Conn_Header_JST_PH_1x02_P2mm_Vertical_SMD"
+		(property "Value" "Solar panel direct solder"
 			(at 194.31 88.9 0)
 			(effects
@@
 			)
 		)
-		(property "Footprint" "Connector_PinHeader_1.00mm:PinHeader_1x02_P1.00mm_Vertical"
+		(property "Footprint" "lib:Solar_Notch_Left_1p0x1p5"
 			(at 194.31 95.25 0)
 			(effects
@@
 			)
 		)
-		(property "Datasheet" "https://www.jst-mfg.com/product/pdf/eng/ePH.pdf"
+		(property "Datasheet" ""
 			(at 194.31 95.25 0)
 			(effects
@@
 			)
 		)
-		(property "Description" "Male JST PH 2 pin connector"
+		(property "Description" ""
 			(at 194.31 95.25 0)
 			(effects

Commit message: Refine solar notches and scale assembly from ZachTek photo
Parts:
- J1: footprint lib:Solar_Notch_Right_1p0x1p5 -> lib:Solar_Notch_Right_1p0x2p0
- J2: footprint lib:Solar_Notch_Left_1p0x1p5 -> lib:Solar_Notch_Left_1p0x2p0
Changed lines of the file:
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@@
 			)
 		)
-		(property "Footprint" "lib:Solar_Notch_Right_1p0x1p5"
+		(property "Footprint" "lib:Solar_Notch_Right_1p0x2p0"
 			(at 194.31 105.41 0)
 			(effects
@@
 			)
 		)
-		(property "Footprint" "lib:Solar_Notch_Left_1p0x1p5"
+		(property "Footprint" "lib:Solar_Notch_Left_1p0x2p0"
 			(at 194.31 95.25 0)
 			(effects

Commit message: Refine v1.1 edge routing and header pad rings
Parts:
- J3: footprint Connector_PinHeader_1.00mm:PinHeader_1x07_P1.00mm_Vertical -> lib:Stratolink_Header_Left_1x07_P1p00_D0p50_Pad0p88
- J4: footprint Connector_PinHeader_1.00mm:PinHeader_1x07_P1.00mm_Vertical -> lib:Stratolink_Header_Right_1x07_P1p00_D0p50_Pad0p88
Changed lines of the file:
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@@
 			)
 		)
-		(property "Footprint" "Connector_PinHeader_1.00mm:PinHeader_1x07_P1.00mm_Vertical"
+		(property "Footprint" "lib:Stratolink_Header_Right_1x07_P1p00_D0p50_Pad0p88"
 			(at 52.07 73.66 0)
 			(effects
@@
 			)
 		)
-		(property "Footprint" "Connector_PinHeader_1.00mm:PinHeader_1x07_P1.00mm_Vertical"
+		(property "Footprint" "lib:Stratolink_Header_Left_1x07_P1p00_D0p50_Pad0p88"
 			(at 20.32 73.66 0)
 			(effects
